File: kicad/voltage-blaster.kicad_pcb (KiCad board)
At the start: 2 copper layers, 95.2 x 24.1 mm, 6 parts, among them J1 Bus_ISA_8bit, U1 LM7905

Commit message: Set PCB revision to 1.1
Other:
- board text added: "rev 1.1"
- board text removed: "rev 2.0"
Changed lines of the file:
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@@
     (title "Voltage Blaster")
     (date 2021-05-23)
-    (rev 2.0)
+    (rev 1.1)
     (company "PhilsComputerLab & Necroware")
     (comment 1 "by Scorp")
@@
     (effects (font (size 1.9 1.9) (thickness 0.4)) (justify mirror))
   )
-  (gr_text "rev 2.0" (at 75.565 61.595) (layer F.SilkS)
+  (gr_text "rev 1.1" (at 75.565 61.595) (layer F.SilkS)
     (effects (font (size 1.2 1.2) (thickness 0.15)))
   )
